File: KiCad/MatrixDisplay/MatrixDisplay-2-sided.kicad_pcb (KiCad board)
At the start: 2 copper layers, 3 parts, among them J1 PUT_IN, J2 Power, U1 mini_esp32

Commit message: minor refactoring
Routing:
- net Net-(U1-Pad18): track 72.2 -> 93.0 mm, vias 0 -> 1
- net Net-(U1-Pad20): track 59.2 -> 70.1 mm, vias 0 -> 1
- net Net-(J1-Pad16): track 49.1 -> 57.5 mm, vias 0 -> 1
- net Net-(J1-Pad7): track 49.0 -> 56.6 mm, vias 0 -> 1
- net Net-(J1-Pad10): track 30.0 -> 35.4 mm, vias 0 -> 1
- net Net-(J1-Pad2): track 18.8 -> 24.0 mm, vias 0 -> 1
- net Net-(J1-Pad8): track 27.2 -> 31.6 mm, vias 0 -> 1
- net Net-(J2-Pad1): track 33.3 -> 37.5 mm
- net Net-(J1-Pad5): track 41.9 -> 45.9 mm, vias 0 -> 1
- net Net-(U1-Pad13): track 41.3 -> 44.4 mm, vias 0 -> 1
- net Net-(J1-Pad6): track 24.4 -> 27.4 mm, vias 0 -> 1
- net Net-(J1-Pad12): track 23.5 -> 25.9 mm, vias 0 -> 1
- net Net-(J1-Pad3): track 34.3 -> 36.4 mm, vias 0 -> 1
- net Net-(J1-Pad1): track 23.4 -> 25.1 mm, vias 0 -> 1
- net Net-(J1-Pad14): track 20.7 -> 20.3 mm, vias 0 -> 1
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